Commit message: update urdf with actual car measurements

File: description/robot.urdf.xacro (robot description, xacro)
@@ -2,3 +2,4 @@
 <robot xmlns:xacro="http://www.ros.org/wiki/xacro"  name="robot">
     <xacro:include filename='robot_core.xacro'/>
+    <xacro:include filename='inertial_macros.xacro'/>
 </robot>

File: description/robot_core.xacro (robot description, xacro)
@@ -1,4 +1,5 @@
 <?xml version="1.0"?>
 <robot xmlns:xacro="http://www.ros.org/wiki/xacro"  name="robot">
+    <xacro:include filename='inertial_macros.xacro'/>
     <material name="grey">
         <color rgba="0.2 0.2 0.2 1"/>
@@ -16,71 +17,74 @@
         <color rgba="0 0 0 1"/>
     </material>
-    <link name="base_link"></link>
+    <link name="base_link">
+    </link>
     <!-- Chassis Link -->
     <joint name="chassis_joint" type="fixed">
         <parent link="base_link"/>
         <child link="chassis"/>
-        <origin xyz="-0.1 0 0"/>
+        <origin xyz="0 0 0"/>
     </joint>
     <link name="chassis">
         <visual>
-            <origin xyz="0.15 0 0.075"/>
+            <origin xyz="0.0 0 0.034925"/> <!--shift the wheels forward half the length of the box-->
             <geometry>
-                <box size="0.3 0.3 0.15"/>
+                <box size="0.232 0.111 0.0635"/> <!--chassis is .232m x .111m x .0635m xyz-->
             </geometry>
             <material name="white"/>
         </visual>
         <collision>
-            <origin xyz="0.15 0 0.075"/>
+            <origin xyz="-0.116 0 0.034925"/>
             <geometry>
-                <box size="0.3 0.3 0.15"/>
+                <box size="0.232 0.111 0.0635"/>
             </geometry>
         </collision>
-        <xacro:inertial_box mass="0.5" x="0.3" y="0.3" z="0.15">
-            <origin xyz="0.15 0 0.075" rpy="0 0 0"/>
+        <xacro:inertial_box mass="0.5" x="0.232" y="0.111" z="0.0635">
+            <origin xyz="-0.116 0 0.034925" rpy="0 0 0"/>
         </xacro:inertial_box>
     </link>
     <!-- Left Wheel -->
-    <joint name="left_wheel" type="continuous">
+    <joint name="left_wheel_joint" type="continuous">
         <parent link="base_link"/>
         <child link="left_wheel"/>
-        <origin xyz="0 0.175 0" rpy="${pi/2} 0 0 "/>
-        <axis xyz="0 0 1"/>
+        <origin xyz="0.058 0.056 0" rpy="${pi/2} 0 0 "/>
+        <axis xyz="0.058 0 1"/>
     </joint>
     <link name="left_wheel">
         <visual>
             <geometry>
-                <cylinder radius="0.5" length="0.04"/>
+                <cylinder radius="0.034925" length="0.0254"/>
             </geometry>
+            <material name="blue"/>
         </visual>
         <collision>
             <geometry>
-                <cylinder radius="0.5" length="0.04"/>
+                <cylinder radius="0.034925" length="0.0254"/>
             </geometry>
         </collision>
-        <xacro:inertial_cylinder mass="0.1" length="0.04" radius="0.05">
-            <origin xyz="0 0 0" rpy="0 0 0"/>
+        <xacro:inertial_cylinder mass="0.1" length="0.0254" radius="0.034925">
+            <origin xyz="0.058 0.056 0" rpy="0 0 0"/>
         </xacro:inertial_cylinder>
     </link>
     <!-- Right Wheel -->
-    <joint name="right_wheel" type="continuous">
+    <joint name="right_wheel_joint" type="continuous">
         <parent link="base_link"/>
         <child link="right_wheel"/>
-        <origin xyz="0 -0.175 0" rpy="${pi/2} 0 0 "/>
-        <axis xyz="0 0 -1"/>
+        <origin xyz="0.058 -0.0556 0" rpy="${pi/2} 0 0 "/>
+        <axis xyz="0.058 0 -1"/>
     </joint>
     <link name="right_wheel">
         <visual>
             <geometry>
-                <cylinder radius="0.5" length="0.04"/>
+                <cylinder radius="0.034925" length="0.0254"/>
             </geometry>
+            <material name="orange"/>
         </visual>
         <collision>
             <geometry>
-                <cylinder radius="0.5" length="0.04"/>
+                <cylinder radius="0.034925" length="0.0254"/>
             </geometry>
         </collision>
-        <xacro:inertial_cylinder mass="0.1" length="0.04" radius="0.05">
-            <origin xyz="0 0 0" rpy="0 0 0"/>
+        <xacro:inertial_cylinder mass="0.1" length="0.0254" radius="0.034925">
+            <origin xyz="0.058 0.056 0" rpy="0 0 0"/>
         </xacro:inertial_cylinder>
     </link>
@@ -89,10 +93,10 @@
         <parent link="chassis"/>
         <child link="caster_wheel"/>
-        <origin xyz="0.24 0 0"/>
+        <origin xyz="-0.058 0 0"/>
     </joint>
     <link name="caster_wheel">
         <visual>
             <geometry>
-                <sphere radius="0.05"/>
+                <sphere radius="0.034925"/>
             </geometry>
             <material name="black"/>
@@ -100,8 +104,8 @@
         <collision>
             <geometry>
-                <sphere radius="0.05"/>
+                <sphere radius="0.034925"/>
             </geometry>
         </collision>
-        <xacro:inertial_sphere mass="0.1" radius="0.05">
+        <xacro:inertial_sphere mass="0.1" radius="0.034925">
             <origin xyz="0 0 0" rpy="0 0 0"/>
         </xacro:inertial_sphere>
