Commit message: update parameters and launch files to get gazebo working

File: description/gazebo_control.xacro (robot description, xacro)
@@ -3,12 +3,21 @@
     <gazebo>
         <plugin name='diff_drive' filename='libgazebo_ros_diff_drive.so'>
+        <ros>
+            <namespace>/</namespace>
+            <argument>--ros-args --remap cmd_vel:=cmd_vel</argument>
+            <argument>--ros-args --remap odom:=odom </argument>
+            <update_rate>10.0</update_rate>
+        </ros>
         <!-- Wheel Info -->
         <left_joint>left_wheel_joint</left_joint>
         <right_joint>right_wheel_joint</right_joint>
-        <wheel_separation>0.127</wheel_separation>
-        <wheel_diameter>0.1</wheel_diameter>
+        <wheel_separation>0.14</wheel_separation> <!--Yellow Wheels-->
+        <wheel_diameter>0.1</wheel_diameter> <!--Yellow Wheels-->
         <!-- Limits -->
         <max_wheel_torque>200</max_wheel_torque>
         <max_wheel_acceleration>10.0</max_wheel_acceleration>
+        <!-- Topics -->
+        <!--odometryTopic>odom</odometryTopic>
+        <commandTopic>cmd_vel</commandTopic-->
         <!-- Output -->
         <odometry_frame>odom</odometry_frame>
@@ -17,4 +26,14 @@
         <publish_odom_tf>true</publish_odom_tf>
         <publish_wheel_tf>true</publish_wheel_tf>
+        <publish_wheel_joint_state>true</publish_wheel_joint_state>
+        </plugin>
+        <plugin name="gazebo_ros_joint_state_publisher" filename="libgazebo_ros_joint_state_publisher.so">
+            <ros>
+                <namespace>/</namespace>
+                <argument>--ros-args --remap joint_states:=joint_states</argument>
+            </ros>
+            <update_rate>100</update_rate>
+            <joint_name>left_wheel_joint</joint_name>
+            <joint_name>right_wheel_joint</joint_name>
         </plugin>
     </gazebo>

File: description/robot.urdf.xacro (robot description, xacro)
@@ -2,4 +2,4 @@
 <robot xmlns:xacro="http://www.ros.org/wiki/xacro"  name="robot">
     <xacro:include filename='robot_core.xacro'/>
-    <xacro:include filename='inertial_macros.xacro'/>
+    <xacro:include filename='gazebo_control.xacro'/>
 </robot>

File: description/robot_core.xacro (robot description, xacro)
@@ -1,19 +1,20 @@
 <?xml version="1.0"?>
 <robot xmlns:xacro="http://www.ros.org/wiki/xacro"  name="robot">
-    <xacro:include filename='inertial_macros.xacro'/>
-    <xacro:property name='chassis_length' value='.232'/>
-    <xacro:property name='chassis_width' value='.111'/>
-    <xacro:property name='chassis_height' value='.064'/>
-    <xacro:property name='chassis_mass' value='.5'/>
-    <xacro:property name='wheel_radius' value='.033'/>
-    <xacro:property name='wheel_thickness' value='.026'/>
-    <xacro:property name='wheel_mass' value='.05'/>
-    <xacro:property name='wheel_offset_x' value='.077'/>
-    <xacro:property name='wheel_offset_y' value='.056'/>
-    <xacro:property name='wheel_offset_z' value='.01'/>
-    <xacro:property name='caster_wheel_radius' value='.01'/>
-    <xacro:property name='caster_wheel_mass' value='.01'/>
-    <xacro:property name='caster_wheel_offset_x' value='.154'/>
-    <xacro:property name='caster_wheel_offset_z' value='${wheel_offset_z - wheel_radius + caster_wheel_radius}'/>
+    <xacro:include filename="inertial_macros.xacro"/>
+    <!-- Car Dimensions -->
+    <xacro:property name="chassis_length" value=".232"/>
+    <xacro:property name="chassis_width" value=".111"/>
+    <xacro:property name="chassis_height" value=".064"/>
+    <xacro:property name="chassis_mass" value=".125"/>
+    <xacro:property name="wheel_radius" value=".04"/>
+    <xacro:property name="wheel_thickness" value=".026"/>
+    <xacro:property name="wheel_mass" value=".05"/>
+    <xacro:property name="wheel_offset_x" value=".058"/>
+    <xacro:property name="wheel_offset_y" value=".07"/>
+    <xacro:property name="wheel_offset_z" value=".01"/>
+    <xacro:property name="caster_wheel_radius" value=".025"/>
+    <xacro:property name="caster_wheel_mass" value=".01"/>
+    <xacro:property name="caster_wheel_offset_x" value=".174"/>
+    <xacro:property name="caster_wheel_offset_z" value="${wheel_offset_z - wheel_radius + caster_wheel_radius}"/>
     <material name="grey">
         <color rgba="0.2 0.2 0.2 1"/>
@@ -31,11 +32,21 @@
         <color rgba="0 0 0 1"/>
     </material>
+    <material name="red">
+        <color rgba="1 0 0 1"/>
+    </material>
     <link name="base_link">
     </link>
+    <link name="odom">
+    </link>
+    <joint name="base_to_odom" type="fixed">
+        <parent link="base_link"/>
+        <child link="odom"/>
+        <origin xyz="0 0 0"/>
+    </joint>
     <!-- Chassis Link -->
     <joint name="chassis_joint" type="fixed">
         <parent link="base_link"/>
         <child link="chassis"/>
-        <origin xyz="${wheel_offset_x} 0 ${-wheel_offset_z}"/>
+        <origin xyz="${-wheel_offset_x} 0 ${-wheel_offset_z}"/>
     </joint>
     <link name="chassis">
@@ -57,5 +68,5 @@
         </xacro:inertial_box>
     </link>
-    <gazebo reference='chassis'>
+    <gazebo reference="chassis">
         <material>Gazebo/White</material>
     </gazebo>
@@ -64,5 +75,5 @@
         <parent link="base_link"/>
         <child link="left_wheel"/>
-        <origin xyz="0 ${wheel_offset_y} 0" rpy="${pi/2} 0 0 "/>
+        <origin xyz="0 ${wheel_offset_y} 0" rpy="-${pi/2} 0 0"/>
         <axis xyz="0 0 1"/>
     </joint>
@@ -77,4 +88,5 @@
             <geometry>
                 <cylinder radius="${wheel_radius}" length="${wheel_thickness}"/>
+                <!--sphere radius="${wheel_radius}"/-->
             </geometry>
         </collision>
@@ -83,6 +95,11 @@
         </xacro:inertial_cylinder>
     </link>
-    <gazebo reference='left_wheel'>
+    <gazebo reference="left_wheel">
         <material>Gazebo/Blue</material>
+        <mu1>0.8</mu1>
+        <mu2>0.8</mu2>
+        <minDepth>0.001</minDepth>
+        <kp>1000000.0</kp>
+        <kd>1.0</kd>
     </gazebo>
     <!-- Right Wheel -->
@@ -90,5 +107,5 @@
         <parent link="base_link"/>
         <child link="right_wheel"/>
-        <origin xyz="0 ${-wheel_offset_y} 0" rpy="${-pi/2} 0 0 "/>
+        <origin xyz="0 ${-wheel_offset_y} 0" rpy="${pi/2} 0 0"/>
         <axis xyz="0 0 -1"/>
     </joint>
@@ -103,4 +120,5 @@
             <geometry>
                 <cylinder radius="${wheel_radius}" length="${wheel_thickness}"/>
+                <!--sphere radius="${wheel_radius}"/-->
             </geometry>
         </collision>
@@ -109,6 +127,11 @@
         </xacro:inertial_cylinder>
     </link>
-    <gazebo reference='right_wheel'>
+    <gazebo reference="right_wheel">
         <material>Gazebo/Orange</material>
+        <mu1>0.8</mu1>
+        <mu2>0.8</mu2>
+        <minDepth>0.001</minDepth>
+        <kp>1000000.0</kp>
+        <kd>1.0</kd>
     </gazebo>
     <!-- Caster Wheel Link -->
@@ -134,8 +157,8 @@
         </xacro:inertial_sphere>
     </link>
-    <gazebo reference='caster_wheel'>
+    <gazebo reference="caster_wheel">
         <material>Gazebo/Black</material>
-        <mu1 value='0.001'/>
-        <mu2 value='0.001'/>
+        <mu1 value="0.001"/>
+        <mu2 value="0.001"/>
     </gazebo>
 </robot>
