Commit message: updates to get lidar simulation working

File: description/lidar.xacro (robot description, xacro)
@@ -10,5 +10,5 @@
         <visual>
             <geometry>
-                <cylinder radius="0.05" length="0.04"/>
+                <cylinder radius="0.025" length="0.04"/>
             </geometry>
         </visual>
@@ -29,5 +29,6 @@
         <sensor name="laser" type="ray">
             <pose> 0 0 0 0 0 0 </pose>
-            <update_rate>10</update_rate>
+            <visualize>true</visualize>
+            <update_rate>40</update_rate>
             <ray>
                 <scan>
@@ -45,4 +46,6 @@
             <plugin name="laser_controller" filename="libgazebo_ros_ray_sensor.so">
                 <ros>
+                    <argument>--ros-args</argument>
+                    <argument>--remap</argument>
                     <argument>~/out:=scan</argument>
                 </ros>

File: description/robot_core.xacro (robot description, xacro)
@@ -31,7 +31,4 @@
     <material name="black">
         <color rgba="0 0 0 1"/>
-    </material>
-    <material name="red">
-        <color rgba="1 0 0 1"/>
     </material>
     <link name="base_link">
